File: old_central_hub/445project_hub.sch (KiCad schematic (older format))
At the start: 56 parts, among them J101 Barrel_Jack_Switch, J102 USB_B, J103 USB, J104 USB, SW101 SW_Push, U101 MCP1826S, U102 SN75240, U103 TUSB2077A, U104 SN75240, U105 SN75240, Y101 6MHz

Commit message: Central Hub rev. 1.1
Parts:
- J101: footprint Connector_BarrelJack:BarrelJack_CUI_PJ-102AH_Horizontal -> Connector_BarrelJack:BarrelJack_Horizontal
- J102: symbol 445project_hub-rescue:USB_B-Connector -> 445project_hub-rescue:USB_B-Connector-445project_hub-rescue
- U103: symbol 445project_hub-rescue:TUSB2077A-tusb2077a -> 445project_hub-rescue:TUSB2077A-tusb2077a-445project_hub-rescue
Connections:
- net +3V3: now also U103.10 (/BUSPWR)
- net GND: no longer U103.10 (/BUSPWR)
Changed lines of the file:
@@
 $EndDescr
 $Comp
-L 445project_hub-rescue:TUSB2077A-tusb2077a U103
+L 445project_hub-rescue:TUSB2077A-tusb2077a-445project_hub-rescue U103
 U 1 1 616349AA
 P 4100 3900
@@
 $EndComp
 $Comp
-L 445project_hub-rescue:USB_B-Connector J102
+L 445project_hub-rescue:USB_B-Connector-445project_hub-rescue J102
 U 1 1 6163E889
 P 1300 2500
@@
 	4100 2150 3950 2150
 Wire Wire Line
-	3950 2150 2950 2150
+	3950 2150 3400 2150
 Wire Wire Line
 	2950 2150 2950 1350
@@
 F 0 "J101" H 1057 4217 50  0000 C CNN
 F 1 "Barrel_Jack_Switch" H 1057 4126 50  0000 C CNN
-F 2 "Connector_BarrelJack:BarrelJack_CUI_PJ-102AH_Horizontal" H 1050 3860 50  0001 C CNN
+F 2 "Connector_BarrelJack:BarrelJack_Horizontal" H 1050 3860 50  0001 C CNN
 F 3 "~" H 1050 3860 50  0001 C CNN
 	1    1000 3900
@@
 	1    0    0    -1
 $EndComp
-Wire Wire Line
-	3550 3300 3300 3300
-Wire Wire Line
-	3300 3300 3300 3700
-Connection ~ 3300 3700
 Wire Wire Line
 	3550 5000 2950 5000
@@
 	1    0    0    -1
 $EndComp
+Wire Wire Line
+	3550 3300 3400 3300
+Wire Wire Line
+	3400 3300 3400 2150
+Connection ~ 3400 2150
+Wire Wire Line
+	3400 2150 2950 2150
 $EndSCHEMATC
