File: old_central_hub/file61787B0F.sch (KiCad schematic (older format))
At the start: 49 parts, among them J201 Conn_01x04, J202 Conn_01x04, J203 Conn_02x05_Odd_Even, J204 Conn_02x05_Odd_Even, J205 Conn_01x04, J206 Conn_02x05_Odd_Even, U201 MCP2221AxSL, U202 MCP2221AxSL, U203 MCP2221AxSL

Commit message: Central Hub rev. 1.1
Parts:
- U201, U202, U203: symbol 445project_hub-rescue:MCP2221AxSL-Interface_USB -> 445project_hub-rescue:MCP2221AxSL-Interface_USB-445project_hub-rescue
Changed lines of the file:
@@
 $EndDescr
 $Comp
-L 445project_hub-rescue:MCP2221AxSL-Interface_USB U201
+L 445project_hub-rescue:MCP2221AxSL-Interface_USB-445project_hub-rescue U201
 U 1 1 617887C4
 P 2200 2300
+AR Path="/617887C4" Ref="U201"  Part="1"
+AR Path="/61787B10/617887C4" Ref="U201"  Part="1"
 F 0 "U201" H 2200 1611 50  0000 C CNN
 F 1 "MCP2221AxSL" H 2200 1520 50  0000 C CNN
@@
 Connection ~ 2200 2900
 $Comp
-L 445project_hub-rescue:MCP2221AxSL-Interface_USB U202
+L 445project_hub-rescue:MCP2221AxSL-Interface_USB-445project_hub-rescue U202
 U 1 1 617C8E19
 P 2900 5800
+AR Path="/617C8E19" Ref="U202"  Part="1"
+AR Path="/61787B10/617C8E19" Ref="U202"  Part="1"
 F 0 "U202" H 2900 5111 50  0000 C CNN
 F 1 "MCP2221AxSL" H 2900 5020 50  0000 C CNN
@@
 Connection ~ 1600 2950
 $Comp
-L 445project_hub-rescue:MCP2221AxSL-Interface_USB U203
+L 445project_hub-rescue:MCP2221AxSL-Interface_USB-445project_hub-rescue U203
 U 1 1 6183F789
 P 6900 3900
+AR Path="/6183F789" Ref="U203"  Part="1"
+AR Path="/61787B10/6183F789" Ref="U203"  Part="1"
 F 0 "U203" H 6900 3211 50  0000 C CNN
 F 1 "MCP2221AxSL" H 6900 3120 50  0000 C CNN
