File: 445project_hub_new.kicad_pcb (KiCad board)
At the start: 2 copper layers, 100 x 100 mm, 116 parts, among them J101 Barrel_Jack_Switch, J102 USB_C_Receptacle_USB2.0, J104 USB, J201 Conn_01x04, J202 Conn_01x04, J203 Conn_02x05_Odd_Even, J204 Conn_02x05_Odd_Even, J205 Conn_01x04, J206 Conn_02x05_Odd_Even, J301 Conn_02x06_Odd_Even, J302 Conn_01x10, J303 Conn_01x04, SW101 SW_Push, U101 MCP1826S, U102 SN75240, U103 TUSB2046I, U104 TPS54302, U105 SN75240, U201 MCP2221AxSL, U202 MCP2221AxSL, U203 MCP2221AxSL, U301 MCP7940N-xSN, U302 MCP23017_SO, U303 DS2482-100, Y101 6MHz, Y301 Crystal

Commit message: Central Hub revision 2.3
Parts:
- added D302: BAT54S, Package_TO_SOT_SMD:SOT-23, F.Cu at (113.6, 78.5)
- added R302: R, Resistor_SMD:R_0603_1608Metric, B.Cu at (116.2, 81.0)
- added U304: DS18B20, Package_TO_SOT_THT:TO-92_Inline, F.Cu at (111.5, 55.5)
Routing:
- net +5V: track 432.0 -> 470.0 mm, vias 2 -> 3
- net Net-(J303-Pad3): track 22.9 -> 35.4 mm
- net Net-(D302-Pad2): track 0.00 -> 3.27 mm, vias 0 -> 1
- net Net-(BT301-Pad1): track 14.2 -> 16.5 mm
- net MCP2221A_VDD: track 314.0 -> 315.4 mm
Other:
- board text added: "Rev. 2.3 20250727"
- board text removed: "Rev. 2.2 20250316"
