File: file61914CDA.kicad_sch (KiCad schematic)
At the start: 14 parts, among them J301 Conn_02x06_Odd_Even, J302 Conn_01x10, J303 Conn_01x04, U301 MCP7940N-xSN, U302 MCP23017_SO, U303 DS2482-100, Y301 Crystal

Commit message: Central Hub revision 2.3
Parts:
- added D302: BAT54S, Package_TO_SOT_SMD:SOT-23, symbol Diode:BAT54S
- added R302: R, Resistor_SMD:R_0603_1608Metric, symbol Device:R
- added U304: DS18B20, Package_TO_SOT_THT:TO-92_Inline, symbol Sensor_Temperature:DS18B20
Connections:
- net GND: now also U304.1 (GND)
- net MCP2221A_VDD: now also D302.3, U304.3 (VDD)
- net at J303.3 (Pin_3), U303.2 (IO): now also U304.2 (DQ)
- net at BT301.1 (+), U301.3 (VBAT): now also R302.2
- new net: D302.2, R302.1
Changed lines of the file:
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@@
   (junction (at 90.17 109.22) (diameter 0) (color 0 0 0 0)
   )
+  (junction (at 162.56 62.23) (diameter 0) (color 0 0 0 0)
+  )
   (junction (at 67.31 54.61) (diameter 0) (color 0 0 0 0)
   )
+  (junction (at 167.64 77.47) (diameter 0) (color 0 0 0 0)
+  )
   (junction (at 121.92 109.22) (diameter 0) (color 0 0 0 0)
   )
+  (junction (at 110.49 26.67) (diameter 0) (color 0 0 0 0)
+  )
   (junction (at 69.85 95.25) (diameter 0) (color 0 0 0 0)
   )
@@
     (stroke (width 0) (type default) (color 0 0 0 0))
   )
+  (wire (pts (xy 179.07 55.88) (xy 167.64 55.88))
+    (stroke (width 0) (type default) (color 0 0 0 0))
+  )
   (wire (pts (xy 127 133.35) (xy 127 129.54))
     (stroke (width 0) (type default) (color 0 0 0 0))
@@
     (stroke (width 0) (type default) (color 0 0 0 0))
   )
+  (wire (pts (xy 167.64 55.88) (xy 167.64 77.47))
+    (stroke (width 0) (type default) (color 0 0 0 0))
+  )
   (wire (pts (xy 72.39 157.48) (xy 72.39 165.1))
     (stroke (width 0) (type default) (color 0 0 0 0))
@@
     (stroke (width 0) (type default) (color 0 0 0 0))
   )
+  (wire (pts (xy 88.9 31.75) (xy 95.25 31.75))
+    (stroke (width 0) (type default) (color 0 0 0 0))
+  )
   (wire (pts (xy 106.68 69.85) (xy 118.11 69.85))
     (stroke (width 0) (type default) (color 0 0 0 0))
@@
     (stroke (width 0) (type default) (color 0 0 0 0))
   )
+  (wire (pts (xy 162.56 48.26) (xy 162.56 62.23))
+    (stroke (width 0) (type default) (color 0 0 0 0))
+  )
   (wire (pts (xy 124.46 124.46) (xy 124.46 129.54))
     (stroke (width 0) (type default) (color 0 0 0 0))
@@
     (stroke (width 0) (type default) (color 0 0 0 0))
   )
-  (wire (pts (xy 137.16 62.23) (xy 173.99 62.23))
+  (wire (pts (xy 137.16 62.23) (xy 162.56 62.23))
     (stroke (width 0) (type default) (color 0 0 0 0))
   )
@@
     (stroke (width 0) (type default) (color 0 0 0 0))
   )
+  (wire (pts (xy 162.56 62.23) (xy 173.99 62.23))
+    (stroke (width 0) (type default) (color 0 0 0 0))
+  )
   (wire (pts (xy 128.27 163.83) (xy 128.27 157.48))
     (stroke (width 0) (type default) (color 0 0 0 0))
@@
     (stroke (width 0) (type default) (color 0 0 0 0))
   )
+  (wire (pts (xy 186.69 48.26) (xy 162.56 48.26))
+    (stroke (width 0) (type default) (color 0 0 0 0))
+  )
   (wire (pts (xy 107.95 127) (xy 123.19 127))
     (stroke (width 0) (type default) (color 0 0 0 0))
@@
     (stroke (width 0) (type default) (color 0 0 0 0))
   )
-  (wire (pts (xy 88.9 54.61) (xy 88.9 49.53))
+  (wire (pts (xy 88.9 31.75) (xy 88.9 54.61))
     (stroke (width 0) (type default) (color 0 0 0 0))
   )
@@
     (pin "1")
   )
+  (symbol (lib_id "power:GND") (at 186.69 63.5 0) (unit 1)
+    (in_bom yes) (on_board yes) (fields_autoplaced)
+    (property "Reference" "#PWR0308" (id 0) (at 186.69 69.85 0)
+      (effects (font (size 1.27 1.27)) hide)
+    )
+    (property "Value" "GND" (id 1) (at 186.69 68.58 0))
+    (property "Footprint" "" (id 2) (at 186.69 63.5 0)
+      (effects (font (size 1.27 1.27)) hide)
+    )
+    (property "Datasheet" "" (id 3) (at 186.69 63.5 0)
+      (effects (font (size 1.27 1.27)) hide)
+    )
+    (pin "1")
+  )
+  (symbol (lib_id "Device:R") (at 106.68 26.67 90) (unit 1)
+    (in_bom yes) (on_board yes) (fields_autoplaced)
+    (property "Reference" "R302" (id 0) (at 106.68 20.32 90))
+    (property "Value" "R" (id 1) (at 106.68 22.86 90))
+    (property "Footprint" "Resistor_SMD:R_0603_1608Metric" (id 2) (at 106.68 28.448 90)
+      (effects (font (size 1.27 1.27)) hide)
+    )
+    (property "Datasheet" "~" (id 3) (at 106.68 26.67 0)
+      (effects (font (size 1.27 1.27)) hide)
+    )
+    (pin "1")
+    (pin "2")
+  )
+  (symbol (lib_id "Sensor_Temperature:DS18B20") (at 186.69 55.88 0) (mirror y) (unit 1)
+    (in_bom yes) (on_board yes) (fields_autoplaced)
+    (property "Reference" "U304" (id 0) (at 193.04 54.6099 0)
+      (effects (font (size 1.27 1.27)) (justify right))
+    )
+    (property "Value" "DS18B20" (id 1) (at 193.04 57.1499 0)
+      (effects (font (size 1.27 1.27)) (justify right))
+    )
+    (property "Footprint" "Package_TO_SOT_THT:TO-92_Inline" (id 2) (at 212.09 62.23 0)
+      (effects (font (size 1.27 1.27)) hide)
+    )
+    (property "Datasheet" "http://datasheets.maximintegrated.com/en/ds/DS18B20.pdf" (id 3) (at 190.5 49.53 0)
+      (effects (font (size 1.27 1.27)) hide)
+    )
+    (pin "1")
+    (pin "2")
+    (pin "3")
+  )
+  (symbol (lib_id "Diode:BAT54S") (at 95.25 26.67 0) (unit 1)
+    (in_bom yes) (on_board yes) (fields_autoplaced)
+    (property "Reference" "D302" (id 0) (at 95.25 20.32 0))
+    (property "Value" "BAT54S" (id 1) (at 95.25 22.86 0))
+    (property "Footprint" "Package_TO_SOT_SMD:SOT-23" (id 2) (at 97.155 23.495 0)
+      (effects (font (size 1.27 1.27)) (justify left) hide)
+    )
+    (property "Datasheet" "https://www.diodes.com/assets/Datasheets/ds11005.pdf" (id 3) (at 92.202 26.67 0)
+      (effects (font (size 1.27 1.27)) hide)
+    )
+    (pin "1")
+    (pin "2")
+    (pin "3")
+  )
 )
